File: kicad/PowerSystem.sch (KiCad schematic (older format))
At the start: 13 parts, among them U201 LF120ABDT-TR, U202 TPS70933

Commit message: Fixed some issues with the schematic and layout
Parts:
- added D203: D_Schottky, symbol D_Schottky
Connections:
- net UbOut: no longer names the net of C204.1, R204.1, TP201.1, U202.5 (Vout)
- net UbOut: now also D203.2 (A)
- new net 5V: D203.1 (K)
Other:
- note added: "Double check the output of the 3.3V\nand watch out for the voltage drop \non the Schottky."
- note removed: "Change the 2.2uF to a Electrolitic?"
- moved on the sheet: C202, C204, D202, R202, R204, TP201, U202
Changed lines of the file:
@@
 L R R202
 U 1 1 584DB059
-P 3200 3850
-F 0 "R202" V 3280 3850 50  0000 C CNN
-F 1 "0Ω" V 3200 3850 50  0000 C CNN
-F 2 "Resistors_SMD:R_0805" V 3130 3850 50  0001 C CNN
-F 3 "" H 3200 3850 50  0000 C CNN
-	1    3200 3850
+P 3200 4250
+F 0 "R202" V 3280 4250 50  0000 C CNN
+F 1 "0Ω" V 3200 4250 50  0000 C CNN
+F 2 "Resistors_SMD:R_0805" V 3130 4250 50  0001 C CNN
+F 3 "" H 3200 4250 50  0000 C CNN
+	1    3200 4250
 	0    1    1    0
 $EndComp
-Text Label 2300 3550 0    60   ~ 0
+Text Label 2300 3950 0    60   ~ 0
 U+
 $Comp
-L GND #PWR015
+L GND #PWR202
 U 1 1 584DB061
-P 3900 4450
-F 0 "#PWR015" H 3900 4200 50  0001 C CNN
-F 1 "GND" H 3900 4300 50  0000 C CNN
-F 2 "" H 3900 4450 50  0000 C CNN
-F 3 "" H 3900 4450 50  0000 C CNN
-	1    3900 4450
+P 3900 4850
+F 0 "#PWR202" H 3900 4600 50  0001 C CNN
+F 1 "GND" H 3900 4700 50  0000 C CNN
+F 2 "" H 3900 4850 50  0000 C CNN
+F 3 "" H 3900 4850 50  0000 C CNN
+	1    3900 4850
 	1    0    0    -1
 $EndComp
@@
 L C C202
 U 1 1 584DB067
-P 2600 4050
-F 0 "C202" H 2625 4150 50  0000 L CNN
-F 1 "1μF 25V" H 2625 3950 50  0000 L CNN
-F 2 "Capacitors_SMD:C_1210" H 2638 3900 50  0001 C CNN
-F 3 "" H 2600 4050 50  0000 C CNN
-F 4 "Value" H 2600 4050 60  0001 C CNN "MFP"
-F 5 "Value" H 2600 4050 60  0001 C CNN "Conrad-PN"
-F 6 "Value" H 2600 4050 60  0001 C CNN "Digikey-PN"
-	1    2600 4050
+P 2600 4450
+F 0 "C202" H 2625 4550 50  0000 L CNN
+F 1 "1μF 25V" H 2625 4350 50  0000 L CNN
+F 2 "Capacitors_SMD:C_1210" H 2638 4300 50  0001 C CNN
+F 3 "" H 2600 4450 50  0000 C CNN
+F 4 "Value" H 2600 4450 60  0001 C CNN "MFP"
+F 5 "Value" H 2600 4450 60  0001 C CNN "Conrad-PN"
+F 6 "Value" H 2600 4450 60  0001 C CNN "Digikey-PN"
+	1    2600 4450
 	1    0    0    -1
 $EndComp
@@
 L C C204
 U 1 1 584DB06E
-P 4650 4050
-F 0 "C204" H 4675 4150 50  0000 L CNN
-F 1 "1μF 16V" H 4675 3950 50  0000 L CNN
-F 2 "Capacitors_SMD:C_1210" H 4688 3900 50  0001 C CNN
-F 3 "" H 4650 4050 50  0000 C CNN
-F 4 "Value" H 4650 4050 60  0001 C CNN "MFP"
-F 5 "Value" H 4650 4050 60  0001 C CNN "Conrad-PN"
-F 6 "Value" H 4650 4050 60  0001 C CNN "Digikey-PN"
-	1    4650 4050
+P 4650 4450
+F 0 "C204" H 4675 4550 50  0000 L CNN
+F 1 "1μF 16V" H 4675 4350 50  0000 L CNN
+F 2 "Capacitors_SMD:C_1210" H 4688 4300 50  0001 C CNN
+F 3 "" H 4650 4450 50  0000 C CNN
+F 4 "Value" H 4650 4450 60  0001 C CNN "MFP"
+F 5 "Value" H 4650 4450 60  0001 C CNN "Conrad-PN"
+F 6 "Value" H 4650 4450 60  0001 C CNN "Digikey-PN"
+	1    4650 4450
 	1    0    0    -1
 $EndComp
@@
 L LED D202
 U 1 1 584DB076
-P 5250 4500
-F 0 "D202" H 5250 4600 50  0000 C CNN
-F 1 "3V3DC" H 5250 4400 50  0000 C CNN
-F 2 "LEDs:LED_0805" H 5250 4500 50  0001 C CNN
-F 3 "" H 5250 4500 50  0000 C CNN
-	1    5250 4500
+P 5250 4900
+F 0 "D202" H 5250 5000 50  0000 C CNN
+F 1 "3V3DC" H 5250 4800 50  0000 C CNN
+F 2 "LEDs:LED_0805" H 5250 4900 50  0001 C CNN
+F 3 "" H 5250 4900 50  0000 C CNN
+	1    5250 4900
 	0    -1   -1   0
 $EndComp
@@
 L R R204
 U 1 1 584DB07D
-P 5250 4000
-F 0 "R204" V 5330 4000 50  0000 C CNN
-F 1 "660Ω" V 5250 4000 50  0000 C CNN
-F 2 "Resistors_SMD:R_0805" V 5180 4000 50  0001 C CNN
-F 3 "" H 5250 4000 50  0000 C CNN
-	1    5250 4000
-	1    0    0    -1
-$EndComp
-$Comp
-L GND #PWR016
+P 5250 4400
+F 0 "R204" V 5330 4400 50  0000 C CNN
+F 1 "660Ω" V 5250 4400 50  0000 C CNN
+F 2 "Resistors_SMD:R_0805" V 5180 4400 50  0001 C CNN
+F 3 "" H 5250 4400 50  0000 C CNN
+	1    5250 4400
+	1    0    0    -1
+$EndComp
+$Comp
+L GND #PWR204
 U 1 1 584DB084
-P 5250 4900
-F 0 "#PWR016" H 5250 4650 50  0001 C CNN
-F 1 "GND" H 5250 4750 50  0000 C CNN
-F 2 "" H 5250 4900 50  0000 C CNN
-F 3 "" H 5250 4900 50  0000 C CNN
-	1    5250 4900
+P 5250 5300
+F 0 "#PWR204" H 5250 5050 50  0001 C CNN
+F 1 "GND" H 5250 5150 50  0000 C CNN
+F 2 "" H 5250 5300 50  0000 C CNN
+F 3 "" H 5250 5300 50  0000 C CNN
+	1    5250 5300
 	1    0    0    -1
 $EndComp
@@
 L TPS70933 U202
 U 1 1 584DB0C1
-P 3900 3700
-F 0 "U202" H 4150 3350 60  0000 C CNN
-F 1 "TPS70933" H 3900 3700 60  0000 C CNN
-F 2 "tl2c-footprint:TPS70933DBVR" H 3750 3700 60  0001 C CNN
-F 3 "" H 3750 3700 60  0000 C CNN
-F 4 "TPS70933DBVR" H 3900 3700 60  0001 C CNN "MFP"
-F 5 "1261694 - 62" H 3900 3700 60  0001 C CNN "Conrad-PN"
-F 6 "296-35483-1-ND" H 3900 3700 60  0001 C CNN "Digikey-PN"
-	1    3900 3700
+P 3900 4100
+F 0 "U202" H 4150 3750 60  0000 C CNN
+F 1 "TPS70933" H 3900 4100 60  0000 C CNN
+F 2 "tl2c-footprint:TPS70933DBVR" H 3750 4100 60  0001 C CNN
+F 3 "" H 3750 4100 60  0000 C CNN
+F 4 "TPS70933DBVR" H 3900 4100 60  0001 C CNN "MFP"
+F 5 "1261694 - 62" H 3900 4100 60  0001 C CNN "Conrad-PN"
+F 6 "296-35483-1-ND" H 3900 4100 60  0001 C CNN "Digikey-PN"
+	1    3900 4100
 	1    0    0    -1
 $EndComp
@@
 $EndComp
 Wire Wire Line
-	3350 3850 3350 3850
-Wire Wire Line
-	2300 3550 3350 3550
-Wire Wire Line
-	3050 3850 2950 3850
-Wire Wire Line
-	2950 3850 2950 3550
-Connection ~ 2950 3550
-Wire Wire Line
-	3900 4200 3900 4450
-Wire Wire Line
-	2600 3550 2600 3900
-Connection ~ 2600 3550
-Wire Wire Line
-	4450 3550 5850 3550
-Wire Wire Line
-	4650 3550 4650 3900
-Connection ~ 4650 3550
-Wire Wire Line
-	4650 4200 4650 4300
-Wire Wire Line
-	4650 4300 3900 4300
-Connection ~ 3900 4300
-Wire Wire Line
-	2600 4200 2600 4400
-Wire Wire Line
-	2600 4400 3900 4400
-Connection ~ 3900 4400
-Wire Wire Line
-	5250 3550 5250 3850
-Connection ~ 5250 3550
-Wire Wire Line
-	5250 4700 5250 4900
-Wire Wire Line
-	5400 3500 5400 3550
-Connection ~ 5400 3550
-Text HLabel 5850 3550 2    60   Input ~ 0
+	3350 4250 3350 4250
+Wire Wire Line
+	2300 3950 3350 3950
+Wire Wire Line
+	3050 4250 2950 4250
+Wire Wire Line
+	2950 4250 2950 3950
+Connection ~ 2950 3950
+Wire Wire Line
+	3900 4600 3900 4850
+Wire Wire Line
+	2600 3950 2600 4300
+Connection ~ 2600 3950
+Wire Wire Line
+	4650 3950 4650 4300
+Connection ~ 4650 3950
+Wire Wire Line
+	4650 4600 4650 4700
+Wire Wire Line
+	4650 4700 3900 4700
+Connection ~ 3900 4700
+Wire Wire Line
+	2600 4600 2600 4800
+Wire Wire Line
+	2600 4800 3900 4800
+Connection ~ 3900 4800
+Wire Wire Line
+	5250 3950 5250 4250
+Connection ~ 5250 3950
+Wire Wire Line
+	5250 5100 5250 5300
+Wire Wire Line
+	5400 3950 5400 3900
+Connection ~ 5400 3950
+Text HLabel 8400 3950 2    60   Input ~ 0
 UbOut
 Wire Wire Line
@@
 $EndComp
 $Comp
-L GND #PWR017
+L GND #PWR201
 U 1 1 584DD17A
 P 3900 2650
-F 0 "#PWR017" H 3900 2400 50  0001 C CNN
+F 0 "#PWR201" H 3900 2400 50  0001 C CNN
 F 1 "GND" H 3900 2500 50  0000 C CNN
 F 2 "" H 3900 2650 50  0000 C CNN
@@
 $EndComp
 $Comp
-L GND #PWR018
+L GND #PWR203
 U 1 1 584DD971
 P 5250 2650
-F 0 "#PWR018" H 5250 2400 50  0001 C CNN
+F 0 "#PWR203" H 5250 2400 50  0001 C CNN
 F 1 "GND" H 5250 2500 50  0000 C CNN
 F 2 "" H 5250 2650 50  0000 C CNN
@@
 L TEST_1P TP201
 U 1 1 584E2106
-P 5400 3500
-F 0 "TP201" H 5400 3770 50  0000 C CNN
-F 1 "TP3V3" H 5400 3700 50  0000 C CNN
-F 2 "Measurement_Points:Measurement_Point_Round-SMD-Pad_Small" H 5600 3500 50  0001 C CNN
-F 3 "" H 5600 3500 50  0000 C CNN
-	1    5400 3500
+P 5400 3900
+F 0 "TP201" H 5400 4170 50  0000 C CNN
+F 1 "TP3V3" H 5400 4100 50  0000 C CNN
+F 2 "Measurement_Points:Measurement_Point_Round-SMD-Pad_Small" H 5600 3900 50  0001 C CNN
+F 3 "" H 5600 3900 50  0000 C CNN
+	1    5400 3900
 	1    0    0    -1
 $EndComp
@@
 	5250 2100 5250 1950
 Wire Wire Line
-	5250 4150 5250 4300
-Text Notes 3300 1100 0    60   ~ 0
-Change the 2.2uF to a Electrolitic?
+	5250 4550 5250 4700
+$Comp
+L D_Schottky D203
+U 1 1 589A3CBF
+P 6200 3950
+F 0 "D203" H 6200 4050 50  0000 C CNN
+F 1 "D_Schottky" H 6200 3850 50  0000 C CNN
+F 2 "" H 6200 3950 60  0000 C CNN
+F 3 "" H 6200 3950 60  0000 C CNN
+	1    6200 3950
+	-1   0    0    1
+$EndComp
+Wire Wire Line
+	4450 3950 6050 3950
+Wire Wire Line
+	6350 3950 8400 3950
+Wire Wire Line
+	6400 3460 7350 3460
+Wire Wire Line
+	7350 3460 7350 3950
+Connection ~ 7350 3950
+Text HLabel 6400 3460 0    60   Input ~ 0
+5V
+Text Notes 5765 4440 0    60   ~ 0
+Double check the output of the 3.3V\nand watch out for the voltage drop \non the Schottky.
 $EndSCHEMATC

Commit message: Made a correction to a net label
Parts:
- C204: value 1μF 16V -> 2.2μF 16V
- D203: footprint (none) -> Diodes_SMD:D_SMA_Standard
Changed lines of the file:
@@
 U+
 $Comp
-L GND #PWR202
+L GND #PWR016
 U 1 1 584DB061
 P 3900 4850
-F 0 "#PWR202" H 3900 4600 50  0001 C CNN
+F 0 "#PWR016" H 3900 4600 50  0001 C CNN
 F 1 "GND" H 3900 4700 50  0000 C CNN
 F 2 "" H 3900 4850 50  0000 C CNN
@@
 P 4650 4450
 F 0 "C204" H 4675 4550 50  0000 L CNN
-F 1 "1μF 16V" H 4675 4350 50  0000 L CNN
+F 1 "2.2μF 16V" H 4675 4350 50  0000 L CNN
 F 2 "Capacitors_SMD:C_1210" H 4688 4300 50  0001 C CNN
 F 3 "" H 4650 4450 50  0000 C CNN
@@
 $EndComp
 $Comp
-L GND #PWR204
+L GND #PWR017
 U 1 1 584DB084
 P 5250 5300
-F 0 "#PWR204" H 5250 5050 50  0001 C CNN
+F 0 "#PWR017" H 5250 5050 50  0001 C CNN
 F 1 "GND" H 5250 5150 50  0000 C CNN
 F 2 "" H 5250 5300 50  0000 C CNN
@@
 $EndComp
 $Comp
-L GND #PWR201
+L GND #PWR018
 U 1 1 584DD17A
 P 3900 2650
-F 0 "#PWR201" H 3900 2400 50  0001 C CNN
+F 0 "#PWR018" H 3900 2400 50  0001 C CNN
 F 1 "GND" H 3900 2500 50  0000 C CNN
 F 2 "" H 3900 2650 50  0000 C CNN
@@
 $EndComp
 $Comp
-L GND #PWR203
+L GND #PWR019
 U 1 1 584DD971
 P 5250 2650
-F 0 "#PWR203" H 5250 2400 50  0001 C CNN
+F 0 "#PWR019" H 5250 2400 50  0001 C CNN
 F 1 "GND" H 5250 2500 50  0000 C CNN
 F 2 "" H 5250 2650 50  0000 C CNN
@@
 F 0 "D203" H 6200 4050 50  0000 C CNN
 F 1 "D_Schottky" H 6200 3850 50  0000 C CNN
-F 2 "" H 6200 3950 60  0000 C CNN
+F 2 "Diodes_SMD:D_SMA_Standard" H 6200 3950 60  0001 C CNN
 F 3 "" H 6200 3950 60  0000 C CNN
 	1    6200 3950
