File: kicad/tl2c.kicad_pcb (KiCad board)
At the start: 4 copper layers, 120.7 x 127 mm, 92 parts, among them IC101 ATTINY20-X, P101 12VDC, P102 I2C Master, P103 Spare, P104 ISP Header, P105 LED_DRIVER, P106 240VAC, P107 LED_DRIVER, P108 LED_OUT, P301 CONN_PIR_OG, P302 CONN_PIR_EG, P303 CONN_PIR_UG, Q301 IRLML2502, Q302 IRLML2502, Q303 IRLML2502, Q401 IRLML2502, Q402 IRLML2502, Q403 IRLML2502, SW101 TL3315NF160Q, U201 LF120ABDT-TR, U202 TPS70933

Commit message: Fixed some issues with the schematic and layout
Parts:
- removed R102: 330Ω, Resistors_SMD:R_0805
- P104: value ISP Header -> TPI Header
- P106: footprint tl2c-footprint:TERMINAL_BLOCK_2_5MM_5MM -> tl2c-footprint:Spring_Terminal_Block_1_x_2_5mm
- P108: footprint tl2c-footprint:TERMINAL_BLOCK_6_5MM_5MM -> tl2c-footprint:Spring_Terminal_Block_1_x_6_5mm
- R103: value 330Ω -> 0Ω
- moved C203 10.4 mm to (111.8, 163.0), turned to 90 degrees
- moved U201 8.33 mm to (106.5, 156.3), turned to 270 degrees
- moved C201 3.24 mm to (105.3, 166.9)
Connections:
- IC101 pad 2: /GPIO_PB0 -> /CLOCK
- IC101 pad 3: /MOSI -> /DATA
- IC101 pad 5: /MISO -> /GPIO_PB2
- IC101 pad 6: /SCK -> /SCL
- P103 pad 2: /GPIO_PB0 -> /GPIO_PB2
- P104 pad 1: /MISO -> /DATA
- P104 pad 3: /SCK -> /CLOCK
- P104 pad 4: /MOSI -> Net-(P104-Pad4)
- P105 pad 6: /GPIO_PB0 -> /GPIO_PB2
- R103 pad 2: /MOSI -> /DATA
- R105 pad 2: /GPIO_PB0 -> /GPIO_PB2
- TP108 pad 1: /GPIO_PB0 -> /GPIO_PB2
Routing:
- net /GPIO_PB0: track 79.2 -> 0.00 mm, vias 1 -> 0
- net /GPIO_PB2: track 0.00 -> 65.4 mm, vias 0 -> 1
- net /SCK: track 54.5 -> 0.00 mm
- net /DATA: track 0.00 -> 48.4 mm, vias 0 -> 2
- net /MOSI: track 47.7 -> 0.00 mm, vias 1 -> 0
- net /CLOCK: track 0.00 -> 36.9 mm, vias 0 -> 1
- net /MISO: track 32.1 -> 0.00 mm
- net /SCL: track 10.6 -> 34.1 mm
- net /PIR13/U+: track 26.1 -> 29.0 mm, vias 7 -> 8
- net /Power System/U+In: track 17.4 -> 15.2 mm
- net /GPIO_PA6: track 66.4 -> 67.9 mm, vias 2 -> 1
- net Net-(P104-Pad4): track 0.00 -> 1.02 mm
Other:
- board text added: "*"

Commit message: Made a correction to a net label
Parts:
- added D203: D_Schottky, Diodes_SMD:D_SMA_Standard, F.Cu at (106.8, 173.2)
- added P109: 5VDC, Pin_Headers:Pin_Header_Straight_1x02_Pitch2.54mm, F.Cu at (95.5, 146.1)
- C204: value 1μF 16V -> 2.2μF 16V
- P104: footprint Pin_Headers:Pin_Header_Straight_2x03 -> tl2c-footprint:TC2030-IDC-FP_ISP_Connector
- moved P104 4.01 mm to (126.5, 125.5), turned to 180 degrees
- moved TP101 1.15 mm to (137.8, 135.4)
- moved SW101 0.89 mm to (117.5, 126.0)
Connections:
- net /CLOCK renamed /TPICLK
- net /DATA renamed /TPIDATA
- C101 pad 1: /PIR13/Ub+ -> /Power System/5V
- C204 pad 1: /PIR13/Ub+ -> Net-(C204-Pad1)
- IC101 pad 1: /PIR13/Ub+ -> /Power System/5V
- P104 pad 2: /PIR13/Ub+ -> /Power System/5V
- P105 pad 7: /PIR13/Ub+ -> /Power System/5V
- Q301 pad 3: /PIR13/Ub+ -> /Power System/5V
- Q302 pad 3: /PIR13/Ub+ -> /Power System/5V
- Q303 pad 3: /PIR13/Ub+ -> /Power System/5V
- R101 pad 2: /PIR13/Ub+ -> /Power System/5V
- R204 pad 1: /PIR13/Ub+ -> Net-(C204-Pad1)
- TP201 pad 1: /PIR13/Ub+ -> Net-(C204-Pad1)
- U202 pad 5: /PIR13/Ub+ -> Net-(C204-Pad1)
Routing:
- net Net-(C204-Pad1): track 0.00 -> 45.2 mm, vias 0 -> 4
- net /PIR13/Ub+: track 23.0 -> 0.00 mm, vias 8 -> 0
- net /Power System/5V: track 0.00 -> 17.7 mm, vias 0 -> 7
- net /TPICLK: track 36.9 -> 40.9 mm, vias 1 -> 2
- net /~Reset: track 37.4 -> 34.3 mm, vias 1 -> 2
- net /TPIDATA: track 48.4 -> 45.8 mm, vias 2 -> 3
- net GND: track 0.00 -> 2.36 mm, vias 0 -> 1
- net Net-(P104-Pad4): track 1.02 -> 0.00 mm
- added copper zone on Ub+, net /Power System/5V
- removed copper zone on Ub+, net /PIR13/Ub+
Other:
- board text added: "5V ISP"
