File: kicad/Hutschiene/PIR13.sch (KiCad schematic (older format))
At the start: 9 parts, among them Q301 IRLML2502, Q302 IRLML2502, Q303 IRLML2502

Commit message: In preperation for using a stencil - moved most 0805 back from handsolder to normal
Parts:
- R301, R302, R303, R307, R308, R309: footprint Resistors_SMD:R_0805_HandSoldering -> Resistors_SMD:R_0805
Changed lines of the file:
@@
 F 0 "R307" V 2300 2160 50  0000 C CNN
 F 1 "10kΩ" V 2220 2160 50  0000 C CNN
-F 2 "Resistors_SMD:R_0805_HandSoldering" V 2150 2160 50  0001 C CNN
+F 2 "Resistors_SMD:R_0805" V 2150 2160 50  0001 C CNN
 F 3 "" H 2220 2160 50  0000 C CNN
 	1    2220 2160
@@
 F 0 "R301" V 1800 2960 50  0000 C CNN
 F 1 "1kΩ" V 1720 2960 50  0000 C CNN
-F 2 "Resistors_SMD:R_0805_HandSoldering" V 1650 2960 50  0001 C CNN
+F 2 "Resistors_SMD:R_0805" V 1650 2960 50  0001 C CNN
 F 3 "" H 1720 2960 50  0000 C CNN
 	1    1720 2960
@@
 F 0 "R308" V 2300 4060 50  0000 C CNN
 F 1 "10kΩ" V 2220 4060 50  0000 C CNN
-F 2 "Resistors_SMD:R_0805_HandSoldering" V 2150 4060 50  0001 C CNN
+F 2 "Resistors_SMD:R_0805" V 2150 4060 50  0001 C CNN
 F 3 "" H 2220 4060 50  0000 C CNN
 	1    2220 4060
@@
 F 0 "R302" V 1800 4860 50  0000 C CNN
 F 1 "1kΩ" V 1720 4860 50  0000 C CNN
-F 2 "Resistors_SMD:R_0805_HandSoldering" V 1650 4860 50  0001 C CNN
+F 2 "Resistors_SMD:R_0805" V 1650 4860 50  0001 C CNN
 F 3 "" H 1720 4860 50  0000 C CNN
 	1    1720 4860
@@
 F 0 "R309" V 2300 5960 50  0000 C CNN
 F 1 "10kΩ" V 2220 5960 50  0000 C CNN
-F 2 "Resistors_SMD:R_0805_HandSoldering" V 2150 5960 50  0001 C CNN
+F 2 "Resistors_SMD:R_0805" V 2150 5960 50  0001 C CNN
 F 3 "" H 2220 5960 50  0000 C CNN
 	1    2220 5960
@@
 F 0 "R303" V 1800 6760 50  0000 C CNN
 F 1 "1kΩ" V 1720 6760 50  0000 C CNN
-F 2 "Resistors_SMD:R_0805_HandSoldering" V 1650 6760 50  0001 C CNN
+F 2 "Resistors_SMD:R_0805" V 1650 6760 50  0001 C CNN
 F 3 "" H 1720 6760 50  0000 C CNN
 	1    1720 6760

Commit message: More refinements based on the DIN prototype tests
Parts:
- R301, R302, R303, R307, R308, R309: footprint Resistors_SMD:R_0805 -> Resistors_SMD:R_0805_HandSoldering
Changed lines of the file:
@@
 F 0 "R307" V 2300 2160 50  0000 C CNN
 F 1 "10kΩ" V 2220 2160 50  0000 C CNN
-F 2 "Resistors_SMD:R_0805" V 2150 2160 50  0001 C CNN
+F 2 "Resistors_SMD:R_0805_HandSoldering" V 2150 2160 50  0001 C CNN
 F 3 "" H 2220 2160 50  0000 C CNN
 	1    2220 2160
@@
 F 0 "R301" V 1800 2960 50  0000 C CNN
 F 1 "1kΩ" V 1720 2960 50  0000 C CNN
-F 2 "Resistors_SMD:R_0805" V 1650 2960 50  0001 C CNN
+F 2 "Resistors_SMD:R_0805_HandSoldering" V 1650 2960 50  0001 C CNN
 F 3 "" H 1720 2960 50  0000 C CNN
 	1    1720 2960
@@
 F 0 "R308" V 2300 4060 50  0000 C CNN
 F 1 "10kΩ" V 2220 4060 50  0000 C CNN
-F 2 "Resistors_SMD:R_0805" V 2150 4060 50  0001 C CNN
+F 2 "Resistors_SMD:R_0805_HandSoldering" V 2150 4060 50  0001 C CNN
 F 3 "" H 2220 4060 50  0000 C CNN
 	1    2220 4060
@@
 F 0 "R302" V 1800 4860 50  0000 C CNN
 F 1 "1kΩ" V 1720 4860 50  0000 C CNN
-F 2 "Resistors_SMD:R_0805" V 1650 4860 50  0001 C CNN
+F 2 "Resistors_SMD:R_0805_HandSoldering" V 1650 4860 50  0001 C CNN
 F 3 "" H 1720 4860 50  0000 C CNN
 	1    1720 4860
@@
 F 0 "R309" V 2300 5960 50  0000 C CNN
 F 1 "10kΩ" V 2220 5960 50  0000 C CNN
-F 2 "Resistors_SMD:R_0805" V 2150 5960 50  0001 C CNN
+F 2 "Resistors_SMD:R_0805_HandSoldering" V 2150 5960 50  0001 C CNN
 F 3 "" H 2220 5960 50  0000 C CNN
 	1    2220 5960
@@
 F 0 "R303" V 1800 6760 50  0000 C CNN
 F 1 "1kΩ" V 1720 6760 50  0000 C CNN
-F 2 "Resistors_SMD:R_0805" V 1650 6760 50  0001 C CNN
+F 2 "Resistors_SMD:R_0805_HandSoldering" V 1650 6760 50  0001 C CNN
 F 3 "" H 1720 6760 50  0000 C CNN
 	1    1720 6760
