File: kicad/Hutschiene/PIR_Connector.sch (KiCad schematic (older format))
At the start: 6 parts

Commit message: Further work on the redesign
Parts:
- C501, C502, C503: renamed from C?; footprint (none) -> Capacitors_SMD:C_0805
- P501, P502, P503: renamed from P?; footprint (none) -> tl2c-footprint:PCB_Screw_Terminal_Block_5mm_x_3
Changed lines of the file:
@@
 PIR_UG
 $Comp
-L CONN_01X03 P?
+L CONN_01X03 P501
 U 1 1 596CE34C
 P 3350 1470
-F 0 "P?" H 3350 1670 50  0000 C CNN
+F 0 "P501" H 3350 1670 50  0000 C CNN
 F 1 "CONN_PIR_OG" V 3450 1470 50  0000 C CNN
-F 2 "" H 3350 1470 50  0000 C CNN
+F 2 "tl2c-footprint:PCB_Screw_Terminal_Block_5mm_x_3" H 3350 1470 50  0001 C CNN
 F 3 "" H 3350 1470 50  0000 C CNN
 	1    3350 1470
@@
 $EndComp
 $Comp
-L CONN_01X03 P?
+L CONN_01X03 P502
 U 1 1 596CE37D
 P 3360 2870
-F 0 "P?" H 3360 3070 50  0000 C CNN
+F 0 "P502" H 3360 3070 50  0000 C CNN
 F 1 "CONN_PIR_EG" V 3460 2870 50  0000 C CNN
-F 2 "" H 3360 2870 50  0000 C CNN
+F 2 "tl2c-footprint:PCB_Screw_Terminal_Block_5mm_x_3" H 3360 2870 50  0001 C CNN
 F 3 "" H 3360 2870 50  0000 C CNN
 	1    3360 2870
@@
 $EndComp
 $Comp
-L CONN_01X03 P?
+L CONN_01X03 P503
 U 1 1 596CE3AC
 P 3360 4210
-F 0 "P?" H 3360 4410 50  0000 C CNN
+F 0 "P503" H 3360 4410 50  0000 C CNN
 F 1 "CONN_PIR_UG" V 3460 4210 50  0000 C CNN
-F 2 "" H 3360 4210 50  0000 C CNN
+F 2 "tl2c-footprint:PCB_Screw_Terminal_Block_5mm_x_3" H 3360 4210 50  0001 C CNN
 F 3 "" H 3360 4210 50  0000 C CNN
 	1    3360 4210
@@
 $EndComp
 $Comp
-L GNDA #PWR?
+L GNDA #PWR028
 U 1 1 596CE74B
 P 2160 2110
-F 0 "#PWR?" H 2160 1860 50  0001 C CNN
+F 0 "#PWR028" H 2160 1860 50  0001 C CNN
 F 1 "GNDA" H 2160 1960 50  0000 C CNN
 F 2 "" H 2160 2110 50  0000 C CNN
@@
 $EndComp
 $Comp
-L GNDA #PWR?
+L GNDA #PWR029
 U 1 1 596CE78C
 P 2210 3550
-F 0 "#PWR?" H 2210 3300 50  0001 C CNN
+F 0 "#PWR029" H 2210 3300 50  0001 C CNN
 F 1 "GNDA" H 2210 3400 50  0000 C CNN
 F 2 "" H 2210 3550 50  0000 C CNN
@@
 $EndComp
 $Comp
-L GNDA #PWR?
+L GNDA #PWR030
 U 1 1 596CE7BF
 P 2200 4820
-F 0 "#PWR?" H 2200 4570 50  0001 C CNN
+F 0 "#PWR030" H 2200 4570 50  0001 C CNN
 F 1 "GNDA" H 2200 4670 50  0000 C CNN
 F 2 "" H 2200 4820 50  0000 C CNN
@@
 $EndComp
 $Comp
-L C C?
+L C C502
 U 1 1 596CF9A5
 P 1730 1660
-F 0 "C?" H 1755 1760 50  0000 L CNN
+F 0 "C502" H 1755 1760 50  0000 L CNN
 F 1 "100nF 50V" H 1755 1560 50  0000 L CNN
-F 2 "" H 1768 1510 50  0000 C CNN
+F 2 "Capacitors_SMD:C_0805" H 1768 1510 50  0001 C CNN
 F 3 "" H 1730 1660 50  0000 C CNN
 F 4 "Value" H 1730 1660 60  0001 C CNN "MPN"
@@
 $EndComp
 $Comp
-L C C?
+L C C501
 U 1 1 596CFB0E
 P 1710 3130
-F 0 "C?" H 1735 3230 50  0000 L CNN
+F 0 "C501" H 1735 3230 50  0000 L CNN
 F 1 "100nF 50V" H 1735 3030 50  0000 L CNN
-F 2 "" H 1748 2980 50  0000 C CNN
+F 2 "Capacitors_SMD:C_0805" H 1748 2980 50  0001 C CNN
 F 3 "" H 1710 3130 50  0000 C CNN
 F 4 "Value" H 1710 3130 60  0001 C CNN "MPN"
@@
 $EndComp
 $Comp
-L C C?
+L C C503
 U 1 1 596CFB51
 P 1760 4390
-F 0 "C?" H 1785 4490 50  0000 L CNN
+F 0 "C503" H 1785 4490 50  0000 L CNN
 F 1 "100nF 50V" H 1785 4290 50  0000 L CNN
-F 2 "" H 1798 4240 50  0000 C CNN
+F 2 "Capacitors_SMD:C_0805" H 1798 4240 50  0001 C CNN
 F 3 "" H 1760 4390 50  0000 C CNN
 F 4 "Value" H 1760 4390 60  0001 C CNN "MPN"
@@
 $EndComp
 Wire Wire Line
-	1190 1370 1360 1370
+	1190 1370 3150 1370
 Wire Wire Line
-	1360 1370 1730 1370
+	1360 2770 3160 2770
 Wire Wire Line
-	1730 1370 3150 1370
+	1360 4110 3160 4110
 Wire Wire Line
-	1360 2770 1710 2770
-Wire Wire Line
-	1710 2770 3160 2770
-Wire Wire Line
-	1360 4110 1760 4110
-Wire Wire Line
-	1760 4110 3160 4110
-Wire Wire Line
-	2210 2870 2210 3310
-Wire Wire Line
-	2210 3310 2210 3550
+	2210 2870 2210 3550
 Wire Wire Line
 	2160 1470 3150 1470
@@
 	1730 1900 2160 1900
 Wire Wire Line
-	2160 1470 2160 1900
-Wire Wire Line
-	2160 1900 2160 2110
+	2160 1470 2160 2110
 Connection ~ 2160 1900
 Wire Wire Line
@@
 	1760 4720 2200 4720
 Wire Wire Line
-	2200 4210 2200 4720
-Wire Wire Line
-	2200 4720 2200 4820
+	2200 4210 2200 4820
 Connection ~ 2200 4720
 Text HLabel 1190 1370 0    60   Input ~ 0
@@
 Connection ~ 1760 4110
 Wire Wire Line
-	1360 1370 1360 2770
-Wire Wire Line
-	1360 2770 1360 4110
+	1360 1370 1360 4110
 Connection ~ 1360 1370
 Connection ~ 1360 2770

Commit message: Adjusted the size and location of the terminal blocks
Parts:
- P501, P502, P503: footprint tl2c-footprint:PCB_Screw_Terminal_Block_5mm_x_3 -> tl2c-footprint:PCB_Screw_Terminal_Block_5.8mm_x_3
Changed lines of the file:
@@
 F 0 "P501" H 3350 1670 50  0000 C CNN
 F 1 "CONN_PIR_OG" V 3450 1470 50  0000 C CNN
-F 2 "tl2c-footprint:PCB_Screw_Terminal_Block_5mm_x_3" H 3350 1470 50  0001 C CNN
+F 2 "tl2c-footprint:PCB_Screw_Terminal_Block_5.8mm_x_3" H 3350 1470 50  0001 C CNN
 F 3 "" H 3350 1470 50  0000 C CNN
 	1    3350 1470
@@
 F 0 "P502" H 3360 3070 50  0000 C CNN
 F 1 "CONN_PIR_EG" V 3460 2870 50  0000 C CNN
-F 2 "tl2c-footprint:PCB_Screw_Terminal_Block_5mm_x_3" H 3360 2870 50  0001 C CNN
+F 2 "tl2c-footprint:PCB_Screw_Terminal_Block_5.8mm_x_3" H 3360 2870 50  0001 C CNN
 F 3 "" H 3360 2870 50  0000 C CNN
 	1    3360 2870
@@
 F 0 "P503" H 3360 4410 50  0000 C CNN
 F 1 "CONN_PIR_UG" V 3460 4210 50  0000 C CNN
-F 2 "tl2c-footprint:PCB_Screw_Terminal_Block_5mm_x_3" H 3360 4210 50  0001 C CNN
+F 2 "tl2c-footprint:PCB_Screw_Terminal_Block_5.8mm_x_3" H 3360 4210 50  0001 C CNN
 F 3 "" H 3360 4210 50  0000 C CNN
 	1    3360 4210

Commit message: More refinements based on the DIN prototype tests
Parts:
- C501, C502, C503: footprint Capacitors_SMD:C_0805 -> Capacitors_SMD:C_0805_HandSoldering
Changed lines of the file:
@@
 $EndComp
 $Comp
-L GNDA #PWR029
+L GNDA #PWR032
 U 1 1 596CE74B
 P 2160 2110
-F 0 "#PWR029" H 2160 1860 50  0001 C CNN
+F 0 "#PWR032" H 2160 1860 50  0001 C CNN
 F 1 "GNDA" H 2160 1960 50  0000 C CNN
 F 2 "" H 2160 2110 50  0000 C CNN
@@
 $EndComp
 $Comp
-L GNDA #PWR030
+L GNDA #PWR033
 U 1 1 596CE78C
 P 2210 3550
-F 0 "#PWR030" H 2210 3300 50  0001 C CNN
+F 0 "#PWR033" H 2210 3300 50  0001 C CNN
 F 1 "GNDA" H 2210 3400 50  0000 C CNN
 F 2 "" H 2210 3550 50  0000 C CNN
@@
 $EndComp
 $Comp
-L GNDA #PWR031
+L GNDA #PWR034
 U 1 1 596CE7BF
 P 2200 4820
-F 0 "#PWR031" H 2200 4570 50  0001 C CNN
+F 0 "#PWR034" H 2200 4570 50  0001 C CNN
 F 1 "GNDA" H 2200 4670 50  0000 C CNN
 F 2 "" H 2200 4820 50  0000 C CNN
@@
 F 0 "C502" H 1755 1760 50  0000 L CNN
 F 1 "100nF 50V" H 1755 1560 50  0000 L CNN
-F 2 "Capacitors_SMD:C_0805" H 1768 1510 50  0001 C CNN
+F 2 "Capacitors_SMD:C_0805_HandSoldering" H 1768 1510 50  0001 C CNN
 F 3 "" H 1730 1660 50  0000 C CNN
 F 4 "Value" H 1730 1660 60  0001 C CNN "MPN"
@@
 F 0 "C501" H 1735 3230 50  0000 L CNN
 F 1 "100nF 50V" H 1735 3030 50  0000 L CNN
-F 2 "Capacitors_SMD:C_0805" H 1748 2980 50  0001 C CNN
+F 2 "Capacitors_SMD:C_0805_HandSoldering" H 1748 2980 50  0001 C CNN
 F 3 "" H 1710 3130 50  0000 C CNN
 F 4 "Value" H 1710 3130 60  0001 C CNN "MPN"
@@
 F 0 "C503" H 1785 4490 50  0000 L CNN
 F 1 "100nF 50V" H 1785 4290 50  0000 L CNN
-F 2 "Capacitors_SMD:C_0805" H 1798 4240 50  0001 C CNN
+F 2 "Capacitors_SMD:C_0805_HandSoldering" H 1798 4240 50  0001 C CNN
 F 3 "" H 1760 4390 50  0000 C CNN
 F 4 "Value" H 1760 4390 60  0001 C CNN "MPN"
