File: kicad/Hutschiene/tl2c.sch (KiCad schematic (older format))
At the start: 31 parts, among them IC101 ATTINY20-X, P101 12VDC, P102 RJ45, P103 CTL CONN, P104 TPI Header, P105 DRV CONN, P106 240VAC, P107 CTL PWR, P108 UG, P109 5VDC, P110 EG, P111 OG, P112 DRV PWR, SW101 TL3315NF160Q

Commit message: More refinements based on the DIN prototype tests
Parts:
- C101, C102: footprint Capacitors_SMD:C_0805 -> Capacitors_SMD:C_0805_HandSoldering
- D101, D102, D103: footprint LEDs:LED_0805 -> LEDs:LED_0805_HandSoldering
- R101, R103, R104, R105, R106, R107, R108: footprint Resistors_SMD:R_0805 -> Resistors_SMD:R_0805_HandSoldering
Changed lines of the file:
@@
 F 0 "C101" H 2185 6270 50  0000 L CNN
 F 1 "100n 50V" H 1760 6070 50  0000 L CNN
-F 2 "Capacitors_SMD:C_0805" H 2198 6020 50  0001 C CNN
+F 2 "Capacitors_SMD:C_0805_HandSoldering" H 2198 6020 50  0001 C CNN
 F 3 "" H 2160 6170 50  0000 C CNN
 	1    2160 6170
@@
 F 0 "R101" V 1545 3250 50  0000 C CNN
 F 1 "10kΩ" V 1465 3250 50  0000 C CNN
-F 2 "Resistors_SMD:R_0805" V 1395 3250 50  0001 C CNN
+F 2 "Resistors_SMD:R_0805_HandSoldering" V 1395 3250 50  0001 C CNN
 F 3 "" H 1465 3250 50  0000 C CNN
 	1    1465 3250
@@
 F 0 "R103" V 5890 6920 50  0000 C CNN
 F 1 "0Ω" V 5810 6920 50  0000 C CNN
-F 2 "Resistors_SMD:R_0805" V 5740 6920 50  0001 C CNN
+F 2 "Resistors_SMD:R_0805_HandSoldering" V 5740 6920 50  0001 C CNN
 F 3 "" H 5810 6920 50  0000 C CNN
 	1    5810 6920
@@
 F 0 "R104" V 6490 6520 50  0000 C CNN
 F 1 "NOPOP" V 6410 6520 50  0000 C CNN
-F 2 "Resistors_SMD:R_0805" V 6340 6520 50  0001 C CNN
+F 2 "Resistors_SMD:R_0805_HandSoldering" V 6340 6520 50  0001 C CNN
 F 3 "" H 6410 6520 50  0000 C CNN
 	1    6410 6520
@@
 F 0 "R105" V 6490 7020 50  0000 C CNN
 F 1 "NOPOP" V 6410 7020 50  0000 C CNN
-F 2 "Resistors_SMD:R_0805" V 6340 7020 50  0001 C CNN
+F 2 "Resistors_SMD:R_0805_HandSoldering" V 6340 7020 50  0001 C CNN
 F 3 "" H 6410 7020 50  0000 C CNN
 	1    6410 7020
@@
 F 0 "D101" H 3700 4010 50  0000 C CNN
 F 1 "LED_UG" H 3700 3810 50  0000 C CNN
-F 2 "LEDs:LED_0805" H 3700 3910 50  0001 C CNN
+F 2 "LEDs:LED_0805_HandSoldering" H 3700 3910 50  0001 C CNN
 F 3 "" H 3700 3910 50  0000 C CNN
 	1    3700 3910
@@
 F 0 "R106" V 3780 3460 50  0000 C CNN
 F 1 "660Ω" V 3700 3460 50  0000 C CNN
-F 2 "Resistors_SMD:R_0805" V 3630 3460 50  0001 C CNN
+F 2 "Resistors_SMD:R_0805_HandSoldering" V 3630 3460 50  0001 C CNN
 F 3 "" H 3700 3460 50  0000 C CNN
 	1    3700 3460
@@
 F 0 "D102" H 4000 4010 50  0000 C CNN
 F 1 "LED_EG" H 4000 3810 50  0000 C CNN
-F 2 "LEDs:LED_0805" H 4000 3910 50  0001 C CNN
+F 2 "LEDs:LED_0805_HandSoldering" H 4000 3910 50  0001 C CNN
 F 3 "" H 4000 3910 50  0000 C CNN
 	1    4000 3910
@@
 F 0 "R107" V 4080 3460 50  0000 C CNN
 F 1 "660Ω" V 4000 3460 50  0000 C CNN
-F 2 "Resistors_SMD:R_0805" V 3930 3460 50  0001 C CNN
+F 2 "Resistors_SMD:R_0805_HandSoldering" V 3930 3460 50  0001 C CNN
 F 3 "" H 4000 3460 50  0000 C CNN
 	1    4000 3460
@@
 F 0 "D103" H 4300 4010 50  0000 C CNN
 F 1 "LED_OG" H 4300 3810 50  0000 C CNN
-F 2 "LEDs:LED_0805" H 4300 3910 50  0001 C CNN
+F 2 "LEDs:LED_0805_HandSoldering" H 4300 3910 50  0001 C CNN
 F 3 "" H 4300 3910 50  0000 C CNN
 	1    4300 3910
@@
 F 0 "R108" V 4380 3460 50  0000 C CNN
 F 1 "660Ω" V 4300 3460 50  0000 C CNN
-F 2 "Resistors_SMD:R_0805" V 4230 3460 50  0001 C CNN
+F 2 "Resistors_SMD:R_0805_HandSoldering" V 4230 3460 50  0001 C CNN
 F 3 "" H 4300 3460 50  0000 C CNN
 	1    4300 3460
@@
 F 0 "C102" H 1790 4000 50  0000 L CNN
 F 1 "100n 50V" H 1915 3900 50  0000 L CNN
-F 2 "Capacitors_SMD:C_0805" H 1803 3750 50  0001 C CNN
+F 2 "Capacitors_SMD:C_0805_HandSoldering" H 1803 3750 50  0001 C CNN
 F 3 "" H 1765 3900 50  0000 C CNN
 	1    1765 3900

Commit message: In preperation for using a stencil - moved most 0805 back from handsolder to normal
Parts:
- C101, C102: footprint Capacitors_SMD:C_0805_HandSoldering -> Capacitors_SMD:C_0805
- R101, R103, R104, R105: footprint Resistors_SMD:R_0805_HandSoldering -> Resistors_SMD:R_0805
Changed lines of the file:
@@
 F 0 "C101" H 2185 6270 50  0000 L CNN
 F 1 "100n 50V" H 1760 6070 50  0000 L CNN
-F 2 "Capacitors_SMD:C_0805_HandSoldering" H 2198 6020 50  0001 C CNN
+F 2 "Capacitors_SMD:C_0805" H 2198 6020 50  0001 C CNN
 F 3 "" H 2160 6170 50  0000 C CNN
 	1    2160 6170
@@
 F 0 "R101" V 1545 3250 50  0000 C CNN
 F 1 "10kΩ" V 1465 3250 50  0000 C CNN
-F 2 "Resistors_SMD:R_0805_HandSoldering" V 1395 3250 50  0001 C CNN
+F 2 "Resistors_SMD:R_0805" V 1395 3250 50  0001 C CNN
 F 3 "" H 1465 3250 50  0000 C CNN
 	1    1465 3250
@@
 F 0 "R103" V 5890 6920 50  0000 C CNN
 F 1 "0Ω" V 5810 6920 50  0000 C CNN
-F 2 "Resistors_SMD:R_0805_HandSoldering" V 5740 6920 50  0001 C CNN
+F 2 "Resistors_SMD:R_0805" V 5740 6920 50  0001 C CNN
 F 3 "" H 5810 6920 50  0000 C CNN
 	1    5810 6920
@@
 F 0 "R104" V 6490 6520 50  0000 C CNN
 F 1 "NOPOP" V 6410 6520 50  0000 C CNN
-F 2 "Resistors_SMD:R_0805_HandSoldering" V 6340 6520 50  0001 C CNN
+F 2 "Resistors_SMD:R_0805" V 6340 6520 50  0001 C CNN
 F 3 "" H 6410 6520 50  0000 C CNN
 	1    6410 6520
@@
 F 0 "R105" V 6490 7020 50  0000 C CNN
 F 1 "NOPOP" V 6410 7020 50  0000 C CNN
-F 2 "Resistors_SMD:R_0805_HandSoldering" V 6340 7020 50  0001 C CNN
+F 2 "Resistors_SMD:R_0805" V 6340 7020 50  0001 C CNN
 F 3 "" H 6410 7020 50  0000 C CNN
 	1    6410 7020
@@
 F 0 "C102" H 1790 4000 50  0000 L CNN
 F 1 "100n 50V" H 1915 3900 50  0000 L CNN
-F 2 "Capacitors_SMD:C_0805_HandSoldering" H 1803 3750 50  0001 C CNN
+F 2 "Capacitors_SMD:C_0805" H 1803 3750 50  0001 C CNN
 F 3 "" H 1765 3900 50  0000 C CNN
 	1    1765 3900

Commit message: Corrected issues with the connectors - Pushing to OSH Park
Parts:
- P105: footprint Pin_Headers:Pin_Header_Straight_2x05_Pitch2.54mm -> Socket_Strips:Socket_Strip_Straight_2x05_Pitch2.54mm
Changed lines of the file:
@@
 F 0 "P105" H 5900 3810 50  0000 C CNN
 F 1 "DRV CONN" H 5900 3910 50  0000 C CNN
-F 2 "Pin_Headers:Pin_Header_Straight_2x05_Pitch2.54mm" H 5900 3260 50  0001 C CNN
+F 2 "Socket_Strips:Socket_Strip_Straight_2x05_Pitch2.54mm" H 5900 3260 50  0001 C CNN
 F 3 "" H 5900 3260 50  0000 C CNN
 	1    5900 3260

Commit message: Moved the RJ45 for the back-plane placement
Parts:
- D101, D102, D103: symbol LED -> LED-RESCUE-tl2c
Changed lines of the file:
@@
 EESchema Schematic File Version 2
+LIBS:tl2c-rescue
 LIBS:tl2c-symbols
 LIBS:power
@@
 NoConn ~ 2365 3400
 $Comp
-L LED D101
+L LED-RESCUE-tl2c D101
 U 1 1 5856AA32
 P 3700 3910
@@
 $EndComp
 $Comp
-L LED D102
+L LED-RESCUE-tl2c D102
 U 1 1 5856B277
 P 4000 3910
@@
 $EndComp
 $Comp
-L LED D103
+L LED-RESCUE-tl2c D103
 U 1 1 5856B503
 P 4300 3910
