File: kicad/Hutschiene/LED_Driver.sch (KiCad schematic (older format))
At the start: 15 parts, among them Q401 IRLML2502, Q402 IRLML2502, Q403 IRLML2502

Commit message: More refinements based on the DIN prototype tests
Parts:
- added R404, R405, R406: 10kΩ, Resistors_SMD:R_0805_HandSoldering, symbol R
- R401, R402, R403, R407, R408, R409: value 10kΩ -> 0kΩ; footprint Resistors_SMD:R_0805 -> Resistors_SMD:R_0805_HandSoldering
Connections:
- net GNDA: now also R404.1, R405.1, R406.1
- net Relay_EG: now also R405.2
- net Relay_OG: now also R406.2
- net Relay_UG: now also R404.2
Other:
- note removed: "TODO - Add a Pull-down\n"
Changed lines of the file:
@@
 P 4750 2350
 F 0 "R401" V 4830 2350 50  0000 C CNN
-F 1 "10kΩ" V 4750 2350 50  0000 C CNN
-F 2 "Resistors_SMD:R_0805" V 4680 2350 50  0001 C CNN
+F 1 "0kΩ" V 4750 2350 50  0000 C CNN
+F 2 "Resistors_SMD:R_0805_HandSoldering" V 4680 2350 50  0001 C CNN
 F 3 "" H 4750 2350 50  0000 C CNN
 	1    4750 2350
@@
 P 4750 3450
 F 0 "R402" V 4830 3450 50  0000 C CNN
-F 1 "10kΩ" V 4750 3450 50  0000 C CNN
-F 2 "Resistors_SMD:R_0805" V 4680 3450 50  0001 C CNN
+F 1 "0kΩ" V 4750 3450 50  0000 C CNN
+F 2 "Resistors_SMD:R_0805_HandSoldering" V 4680 3450 50  0001 C CNN
 F 3 "" H 4750 3450 50  0000 C CNN
 	1    4750 3450
@@
 P 4750 4500
 F 0 "R403" V 4830 4500 50  0000 C CNN
-F 1 "10kΩ" V 4750 4500 50  0000 C CNN
-F 2 "Resistors_SMD:R_0805" V 4680 4500 50  0001 C CNN
+F 1 "0kΩ" V 4750 4500 50  0000 C CNN
+F 2 "Resistors_SMD:R_0805_HandSoldering" V 4680 4500 50  0001 C CNN
 F 3 "" H 4750 4500 50  0000 C CNN
 	1    4750 4500
@@
 Wire Wire Line
 	5500 3650 5500 3600
-Text Notes 3700 2700 0    60   ~ 0
-TODO - Add a Pull-down\n
 Text HLabel 4200 2350 0    60   Input ~ 0
 Relay_UG
@@
 P 5750 1950
 F 0 "R407" V 5830 1950 50  0000 C CNN
-F 1 "10kΩ" V 5750 1950 50  0000 C CNN
-F 2 "Resistors_SMD:R_0805" V 5680 1950 50  0001 C CNN
+F 1 "0kΩ" V 5750 1950 50  0000 C CNN
+F 2 "Resistors_SMD:R_0805_HandSoldering" V 5680 1950 50  0001 C CNN
 F 3 "" H 5750 1950 50  0000 C CNN
 	1    5750 1950
@@
 P 5750 3050
 F 0 "R408" V 5830 3050 50  0000 C CNN
-F 1 "10kΩ" V 5750 3050 50  0000 C CNN
-F 2 "Resistors_SMD:R_0805" V 5680 3050 50  0001 C CNN
+F 1 "0kΩ" V 5750 3050 50  0000 C CNN
+F 2 "Resistors_SMD:R_0805_HandSoldering" V 5680 3050 50  0001 C CNN
 F 3 "" H 5750 3050 50  0000 C CNN
 	1    5750 3050
@@
 P 5750 4050
 F 0 "R409" V 5830 4050 50  0000 C CNN
-F 1 "10kΩ" V 5750 4050 50  0000 C CNN
-F 2 "Resistors_SMD:R_0805" V 5680 4050 50  0001 C CNN
+F 1 "0kΩ" V 5750 4050 50  0000 C CNN
+F 2 "Resistors_SMD:R_0805_HandSoldering" V 5680 4050 50  0001 C CNN
 F 3 "" H 5750 4050 50  0000 C CNN
 	1    5750 4050
@@
 	5500 1950 5500 2100
 Wire Wire Line
-	4800 5200 4800 4950
-Wire Wire Line
-	4800 4950 4300 4950
-Text HLabel 4300 4950 0    60   Input ~ 0
+	4480 5890 4480 5780
+Wire Wire Line
+	4480 5780 3980 5780
+Text HLabel 3980 5780 0    60   Input ~ 0
 LED_DRIVER_GND
 $Comp
 L GNDA #PWR025
 U 1 1 5856DA15
-P 4800 5200
-F 0 "#PWR025" H 4800 4950 50  0001 C CNN
-F 1 "GNDA" H 4800 5050 50  0000 C CNN
-F 2 "" H 4800 5200 50  0000 C CNN
-F 3 "" H 4800 5200 50  0000 C CNN
-	1    4800 5200
+P 4480 5890
+F 0 "#PWR025" H 4480 5640 50  0001 C CNN
+F 1 "GNDA" H 4480 5740 50  0000 C CNN
+F 2 "" H 4480 5890 50  0000 C CNN
+F 3 "" H 4480 5890 50  0000 C CNN
+	1    4480 5890
 	1    0    0    -1
 $EndComp
@@
 Wire Wire Line
 	4200 2350 4600 2350
+$Comp
+L R R404
+U 1 1 59B97532
+P 4400 2640
+F 0 "R404" V 4480 2640 50  0000 C CNN
+F 1 "10kΩ" V 4400 2640 50  0000 C CNN
+F 2 "Resistors_SMD:R_0805_HandSoldering" V 4330 2640 50  0001 C CNN
+F 3 "" H 4400 2640 50  0000 C CNN
+	1    4400 2640
+	-1   0    0    1
+$EndComp
+$Comp
+L GNDA #PWR029
+U 1 1 59B9770A
+P 4400 2910
+F 0 "#PWR029" H 4400 2660 50  0001 C CNN
+F 1 "GNDA" H 4400 2760 50  0000 C CNN
+F 2 "" H 4400 2910 50  0000 C CNN
+F 3 "" H 4400 2910 50  0000 C CNN
+	1    4400 2910
+	1    0    0    -1
+$EndComp
+Wire Wire Line
+	4400 2350 4400 2490
+Connection ~ 4400 2350
+Wire Wire Line
+	4400 2790 4400 2910
+$Comp
+L R R405
+U 1 1 59B97CA3
+P 4400 3710
+F 0 "R405" V 4480 3710 50  0000 C CNN
+F 1 "10kΩ" V 4400 3710 50  0000 C CNN
+F 2 "Resistors_SMD:R_0805_HandSoldering" V 4330 3710 50  0001 C CNN
+F 3 "" H 4400 3710 50  0000 C CNN
+	1    4400 3710
+	-1   0    0    1
+$EndComp
+$Comp
+L GNDA #PWR030
+U 1 1 59B97CA9
+P 4400 3980
+F 0 "#PWR030" H 4400 3730 50  0001 C CNN
+F 1 "GNDA" H 4400 3830 50  0000 C CNN
+F 2 "" H 4400 3980 50  0000 C CNN
+F 3 "" H 4400 3980 50  0000 C CNN
+	1    4400 3980
+	1    0    0    -1
+$EndComp
+Wire Wire Line
+	4400 3860 4400 3980
+$Comp
+L R R406
+U 1 1 59B9818B
+P 4400 4790
+F 0 "R406" V 4480 4790 50  0000 C CNN
+F 1 "10kΩ" V 4400 4790 50  0000 C CNN
+F 2 "Resistors_SMD:R_0805_HandSoldering" V 4330 4790 50  0001 C CNN
+F 3 "" H 4400 4790 50  0000 C CNN
+	1    4400 4790
+	-1   0    0    1
+$EndComp
+$Comp
+L GNDA #PWR031
+U 1 1 59B98191
+P 4400 5060
+F 0 "#PWR031" H 4400 4810 50  0001 C CNN
+F 1 "GNDA" H 4400 4910 50  0000 C CNN
+F 2 "" H 4400 5060 50  0000 C CNN
+F 3 "" H 4400 5060 50  0000 C CNN
+	1    4400 5060
+	1    0    0    -1
+$EndComp
+Wire Wire Line
+	4400 4940 4400 5060
+Wire Wire Line
+	4400 3450 4400 3560
+Connection ~ 4400 3450
+Wire Wire Line
+	4400 4500 4400 4640
+Connection ~ 4400 4500
 $EndSCHEMATC

Commit message: In preperation for using a stencil - moved most 0805 back from handsolder to normal
Parts:
- R401, R402, R403, R404, R405, R406, R407, R408, R409: footprint Resistors_SMD:R_0805_HandSoldering -> Resistors_SMD:R_0805
Changed lines of the file:
@@
 F 0 "R401" V 4830 2350 50  0000 C CNN
 F 1 "0kΩ" V 4750 2350 50  0000 C CNN
-F 2 "Resistors_SMD:R_0805_HandSoldering" V 4680 2350 50  0001 C CNN
+F 2 "Resistors_SMD:R_0805" V 4680 2350 50  0001 C CNN
 F 3 "" H 4750 2350 50  0000 C CNN
 	1    4750 2350
@@
 F 0 "R402" V 4830 3450 50  0000 C CNN
 F 1 "0kΩ" V 4750 3450 50  0000 C CNN
-F 2 "Resistors_SMD:R_0805_HandSoldering" V 4680 3450 50  0001 C CNN
+F 2 "Resistors_SMD:R_0805" V 4680 3450 50  0001 C CNN
 F 3 "" H 4750 3450 50  0000 C CNN
 	1    4750 3450
@@
 F 0 "R403" V 4830 4500 50  0000 C CNN
 F 1 "0kΩ" V 4750 4500 50  0000 C CNN
-F 2 "Resistors_SMD:R_0805_HandSoldering" V 4680 4500 50  0001 C CNN
+F 2 "Resistors_SMD:R_0805" V 4680 4500 50  0001 C CNN
 F 3 "" H 4750 4500 50  0000 C CNN
 	1    4750 4500
@@
 F 0 "R407" V 5830 1950 50  0000 C CNN
 F 1 "0kΩ" V 5750 1950 50  0000 C CNN
-F 2 "Resistors_SMD:R_0805_HandSoldering" V 5680 1950 50  0001 C CNN
+F 2 "Resistors_SMD:R_0805" V 5680 1950 50  0001 C CNN
 F 3 "" H 5750 1950 50  0000 C CNN
 	1    5750 1950
@@
 F 0 "R408" V 5830 3050 50  0000 C CNN
 F 1 "0kΩ" V 5750 3050 50  0000 C CNN
-F 2 "Resistors_SMD:R_0805_HandSoldering" V 5680 3050 50  0001 C CNN
+F 2 "Resistors_SMD:R_0805" V 5680 3050 50  0001 C CNN
 F 3 "" H 5750 3050 50  0000 C CNN
 	1    5750 3050
@@
 F 0 "R409" V 5830 4050 50  0000 C CNN
 F 1 "0kΩ" V 5750 4050 50  0000 C CNN
-F 2 "Resistors_SMD:R_0805_HandSoldering" V 5680 4050 50  0001 C CNN
+F 2 "Resistors_SMD:R_0805" V 5680 4050 50  0001 C CNN
 F 3 "" H 5750 4050 50  0000 C CNN
 	1    5750 4050
@@
 F 0 "R404" V 4480 2640 50  0000 C CNN
 F 1 "10kΩ" V 4400 2640 50  0000 C CNN
-F 2 "Resistors_SMD:R_0805_HandSoldering" V 4330 2640 50  0001 C CNN
+F 2 "Resistors_SMD:R_0805" V 4330 2640 50  0001 C CNN
 F 3 "" H 4400 2640 50  0000 C CNN
 	1    4400 2640
@@
 F 0 "R405" V 4480 3710 50  0000 C CNN
 F 1 "10kΩ" V 4400 3710 50  0000 C CNN
-F 2 "Resistors_SMD:R_0805_HandSoldering" V 4330 3710 50  0001 C CNN
+F 2 "Resistors_SMD:R_0805" V 4330 3710 50  0001 C CNN
 F 3 "" H 4400 3710 50  0000 C CNN
 	1    4400 3710
@@
 F 0 "R406" V 4480 4790 50  0000 C CNN
 F 1 "10kΩ" V 4400 4790 50  0000 C CNN
-F 2 "Resistors_SMD:R_0805_HandSoldering" V 4330 4790 50  0001 C CNN
+F 2 "Resistors_SMD:R_0805" V 4330 4790 50  0001 C CNN
 F 3 "" H 4400 4790 50  0000 C CNN
 	1    4400 4790

Commit message: Upgrade to KiCad 5.1
Parts:
- D404, D405, D406: symbol D -> Device:D
- Q401, Q402, Q403: symbol IRLML2502 -> tl2c-symbols:IRLML2502
- R401, R402, R403, R404, R405, R406, R407, R408, R409: symbol R -> Device:R
- REL101, REL102, REL103: symbol Relay_JW1AFSN12F -> tl2c-symbols:Relay_JW1AFSN12F
Changed lines of the file:
@@
-EESchema Schematic File Version 2
-LIBS:tl2c-rescue
-LIBS:tl2c-symbols
-LIBS:power
-LIBS:device
-LIBS:transistors
-LIBS:conn
-LIBS:linear
-LIBS:regul
-LIBS:74xx
-LIBS:cmos4000
-LIBS:adc-dac
-LIBS:memory
-LIBS:xilinx
-LIBS:microcontrollers
-LIBS:dsp
-LIBS:microchip
-LIBS:analog_switches
-LIBS:motorola
-LIBS:texas
-LIBS:intel
-LIBS:audio
-LIBS:interface
-LIBS:digital-audio
-LIBS:philips
-LIBS:display
-LIBS:cypress
-LIBS:siliconi
-LIBS:opto
-LIBS:atmel
-LIBS:contrib
-LIBS:valves
+EESchema Schematic File Version 4
 LIBS:tl2c-cache
-EELAYER 25 0
+EELAYER 26 0
 EELAYER END
 $Descr A4 11693 8268
@@
 $EndDescr
 $Comp
-L Relay_JW1AFSN12F REL?
+L tl2c-symbols:Relay_JW1AFSN12F REL?
 U 1 1 5852585A
 P 6450 1950
@@
 $EndComp
 $Comp
-L Relay_JW1AFSN12F REL?
+L tl2c-symbols:Relay_JW1AFSN12F REL?
 U 1 1 58525862
 P 6450 3050
@@
 $EndComp
 $Comp
-L Relay_JW1AFSN12F REL?
+L tl2c-symbols:Relay_JW1AFSN12F REL?
 U 1 1 5852586A
 P 6450 4050
@@
 $EndComp
 $Comp
-L D D404
+L Device:D D404
 U 1 1 58525871
 P 6425 2350
@@
 $EndComp
 $Comp
-L D D405
+L Device:D D405
 U 1 1 58525878
 P 6425 3400
@@
 $EndComp
 $Comp
-L D D406
+L Device:D D406
 U 1 1 5852587F
 P 6425 4400
@@
 $EndComp
 $Comp
-L R R401
+L Device:R R401
 U 1 1 58525889
 P 4750 2350
@@
 $EndComp
 $Comp
-L R R402
+L Device:R R402
 U 1 1 58525890
 P 4750 3450
@@
 $EndComp
 $Comp
-L R R403
+L Device:R R403
 U 1 1 58525897
 P 4750 4500
@@
 $EndComp
 $Comp
-L IRLML2502 Q401
+L tl2c-symbols:IRLML2502 Q401
 U 1 1 5852589F
 P 5400 2300
@@
 $EndComp
 $Comp
-L IRLML2502 Q402
+L tl2c-symbols:IRLML2502 Q402
 U 1 1 585258A7
 P 5400 3400
@@
 $EndComp
 $Comp
-L IRLML2502 Q403
+L tl2c-symbols:IRLML2502 Q403
 U 1 1 585258AF
 P 5400 4450
@@
 LED_DRIVER_U+
 $Comp
-L R R407
+L Device:R R407
 U 1 1 5852702F
 P 5750 1950
@@
 Connection ~ 5950 1950
 $Comp
-L R R408
+L Device:R R408
 U 1 1 585271D4
 P 5750 3050
@@
 Connection ~ 5950 3050
 $Comp
-L R R409
+L Device:R R409
 U 1 1 58527308
 P 5750 4050
@@
 LED_DRIVER_GND
 $Comp
-L GNDA #PWR025
+L power:GNDA #PWR025
 U 1 1 5856DA15
 P 4480 5890
@@
 $EndComp
 $Comp
-L GNDA #PWR026
+L power:GNDA #PWR026
 U 1 1 5856DA56
 P 5500 4800
@@
 $EndComp
 $Comp
-L GNDA #PWR027
+L power:GNDA #PWR027
 U 1 1 5856DA97
 P 5500 3650
@@
 $EndComp
 $Comp
-L GNDA #PWR028
+L power:GNDA #PWR028
 U 1 1 5856DAD8
 P 5500 2600
@@
 	4200 2350 4600 2350
 $Comp
-L R R404
+L Device:R R404
 U 1 1 59B97532
 P 4400 2640
@@
 $EndComp
 $Comp
-L GNDA #PWR029
+L power:GNDA #PWR029
 U 1 1 59B9770A
 P 4400 2910
@@
 	4400 2790 4400 2910
 $Comp
-L R R405
+L Device:R R405
 U 1 1 59B97CA3
 P 4400 3710
@@
 $EndComp
 $Comp
-L GNDA #PWR030
+L power:GNDA #PWR030
 U 1 1 59B97CA9
 P 4400 3980
@@
 	4400 3860 4400 3980
 $Comp
-L R R406
+L Device:R R406
 U 1 1 59B9818B
 P 4400 4790
@@
 $EndComp
 $Comp
-L GNDA #PWR031
+L power:GNDA #PWR031
 U 1 1 59B98191
 P 4400 5060
