File: kicad/Hutschiene/tl2c.kicad_pcb (KiCad board)
At the start: 4 copper layers, 175.9 x 86.5 mm, 92 parts, among them IC101 ATTINY20-X, P101 12VDC, P102 RJ45, P103 CTL CONN, P104 TPI Header, P105 DRV CONN, P106 240VAC, P107 CTL PWR, P108 UG, P109 5VDC, P110 EG, P111 OG, P112 DRV PWR, P201 Mode_Bridge, P501 CONN_PIR_OG, P502 CONN_PIR_EG, P503 CONN_PIR_UG, Q301 IRLML2502, Q302 IRLML2502, Q303 IRLML2502, Q401 IRLML2502, Q402 IRLML2502, Q403 IRLML2502, SW101 TL3315NF160Q, U201 LF120ABDT-TR, U202 TPS70933

Commit message: Updated to release KiCad release 10
Connections:
- net /~Reset renamed /~{Reset}
Routing:
- added copper zone on In2.Cu, net /PIR13/U+
- added copper zone on In1.Cu, net /PIR13/Ub+
- removed copper zone on U+, net /PIR13/U+
- removed copper zone on Ub+, net /PIR13/Ub+
Other:
- net class Default removed
