File: kicad/Controller/tl2c.kicad_pcb (KiCad board)
At the start: 4 copper layers, 120.7 x 127 mm, 95 parts, among them IC101 ATTINY20-X, P101 12VDC, P102 I2C Master, P103 Spare, P104 TPI Header, P105 LED_DRIVER, P106 240VAC, P107 LED_DRIVER, P108 LED_OUT, P109 5VDC, P201 Mode_Bridge, P301 CONN_PIR_OG, P302 CONN_PIR_EG, P303 CONN_PIR_UG, Q301 IRLML2502, Q302 IRLML2502, Q303 IRLML2502, Q401 IRLML2502, Q402 IRLML2502, Q403 IRLML2502, SW101 TL3315NF160Q, U201 LF120ABDT-TR, U202 TPS70933

Commit message: Small changes to the clearances
Other:
- board text added: "Rly Int"
Changed lines of the file:
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@@
     (area 11.304001 32.456 173.659715 192.505001)
     (thickness 1.6)
-    (drawings 116)
+    (drawings 117)
     (tracks 396)
     (zones 0)
@@
       (net 46 "Net-(F101-Pad2)"))
   )
+  (gr_text "Rly\nInt" (at 145.3 131.7) (layer F.SilkS)
+    (effects (font (size 0.762 0.762) (thickness 0.127)))
+  )
   (gr_text "ISP \nPWR" (at 94.869 142.875 90) (layer F.SilkS)

Commit message: Bringing the board into the latest KiCad
Connections:
- net /~Reset renamed /~{Reset}
Routing:
- added copper zone on In2.Cu, net /PIR13/U+
- added copper zone on In1.Cu, net /PIR13/Ub+
- removed copper zone on U+, net /PIR13/U+
- removed copper zone on Ub+, net /PIR13/Ub+
Other:
- net class Default removed
