File: kicad/esp32/Zone_3_Enable.kicad_sch (KiCad schematic)
At the start: 5 parts, among them SW401 B3F-1150

Commit message: Created rev 1.01 - Addes some more labels and annotations
Other:
- title: (none) -> TL2C-ESP32-1 TL2C Adapter for ESP32
Changed lines of the file:
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@@
 	(generator "eeschema")
 	(generator_version "8.0")
-	(paper "A4")
+	(paper "A3")
+	(title_block
+		(title "TL2C-ESP32-1 TL2C Adapter for ESP32")
+		(date "2024-02-08")
+		(rev "1.01")
+	)
 	(junction
 		(at 107.95 62.23)

Commit message: Reseated the RJ45
Parts:
- R401: value 51κΩ -> 47κΩ
- R402: value 21kΩ -> 470Ω
Changed lines of the file:
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@@
 		(dnp no)
 		(property "Reference" "R401"
-			(at 85.09 45.72 0)
+			(at 82.55 45.72 0)
 			(effects
 				(font
@@
 			)
 		)
-		(property "Value" "51κΩ"
+		(property "Value" "47κΩ"
 			(at 82.55 48.26 0)
 			(effects
@@
 			)
 		)
-		(property "Value" "21kΩ"
+		(property "Value" "470Ω"
 			(at 99.06 59.4939 90)
 			(effects

Commit message: R1 correction
Parts:
- R401: value 47κΩ -> 4.7κΩ
Changed lines of the file:
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@@
 			)
 		)
-		(property "Value" "47κΩ"
+		(property "Value" "4.7κΩ"
 			(at 82.55 48.26 0)
 			(effects

Commit message: Adding some documentation
Parts:
- C401: value 1μF -> 0.1μF
Changed lines of the file:
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@@
 		(fields_autoplaced yes)
 		(property "Reference" "C401"
-			(at 112.141 68.6379 0)
+			(at 112.141 68.6378 0)
 			(effects
 				(font
@@
 			)
 		)
-		(property "Value" "1μF"
+		(property "Value" "0.1μF"
 			(at 112.141 71.0621 0)
 			(effects

Commit message: Updated the artwork and documentation
Parts:
- R401: value 4.7κΩ -> 10κΩ
- R402: value 470Ω -> 10κΩ
Changed lines of the file:
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@@
 			)
 		)
-		(property "Value" "4.7κΩ"
+		(property "Value" "10κΩ"
 			(at 82.55 48.26 0)
 			(effects
@@
 		(fields_autoplaced yes)
 		(property "Reference" "R402"
-			(at 99.06 57.0697 90)
-			(effects
-				(font
-					(size 1.27 1.27)
-				)
-			)
-		)
-		(property "Value" "470Ω"
-			(at 99.06 59.4939 90)
-			(effects
-				(font
+			(at 99.06 57.0695 90)
+			(effects
+				(font
+					(size 1.27 1.27)
+				)
+			)
+		)
+		(property "Value" "10κΩ"
+			(at 99.06 59.4938 90)
+			(effects
+				(font
