File: kicad/esp32/esp32.kicad_sch (KiCad schematic)
At the start: 32 parts, among them J101 RJ45, J102 NodeMCU, J103 Annunciator, U101 74LS14, X101 Mouse Bites, X102 Mouse Bites, X103 Mouse Bites, X104 Mouse Bites

Commit message: Updated the artwork and documentation
Parts:
- removed U101: 74LS14, Package_SO:SO-14_5.3x10.2mm_P1.27mm, symbol 74xx:74LS14
- added U101: 74HC14, Package_SO:SO-14_5.3x10.2mm_P1.27mm, symbol 74xx:74HC14
Connections:
- net +3V3: now also U101.14 (VCC)
- net GND: now also U101.7 (GND)
- net ZONE1_BTN: now also U101.2
- net ZONE2_BTN: now also U101.4
- net Zone 1 Enable/ZONE_GPIO: now also U101.1
- net Zone 2 Enable/ZONE_GPIO: now also U101.3
- net Zone 3 Enable/ZONE_GPIO: now also U101.5
