File: kicad/esp32/esp32.kicad_sch (KiCad schematic)
At the start: 32 parts, among them J101 RJ45, J102 NodeMCU, J103 Annunciator, U101 74HC14, X101 Mouse Bites, X102 Mouse Bites, X103 Mouse Bites, X104 Mouse Bites

Commit message: Update and archive for kicad 10.0.2
Parts:
- M101: value ~ -> (none)
Connections:
- net ~{SLEEP}: now also M101.10 (D27); no longer M101.5 (D35)
