File: kicad/esp32/esp32.kicad_pcb (KiCad board)
At the start: 2 copper layers, 67.5 x 102.7 mm, 47 parts, among them J101 RJ45, J102 NodeMCU, J103 Annunciator, SW201 B3F-1150, SW301 B3F-1150, SW401 B3F-1150, U101 74HC14, X101 Mouse Bites, X102 Mouse Bites, X103 Mouse Bites, X104 Mouse Bites

Commit message: Update and archive for kicad 10.0.2
Connections:
- M101 pad 10: unconnected-(M101-D27-Pad10) -> /~{SLEEP}
- M101 pad 5: /~{SLEEP} -> unconnected-(M101-D35-Pad5)
Routing:
- net /~{SLEEP}: track 40.5 -> 29.9 mm
Other:
- board text added: "TL2C-ESP32-1 Rev ${REVISION}"
- board text removed: "TL2C-ESP32-1 Rev 1.10"
